Commit message: hanees hand with a tf

File: advr_mob_plt_description/urdf/main.urdf (robot description, URDF)
Before this commit: robot COVER, 24 links, 23 joints
Links:
- added link footprint
Joints:
- added joint base_joint: type fixed, parent footprint, child 1_A

Commit message: hanes hand test urdf is done till knuckle

File: advr_mob_plt_description/urdf/main.urdf (robot description, URDF)
Before this commit: robot COVER, 25 links, 24 joints
Joints:
- removed joint 1_A--PAF1003901
- removed joint 1_A--PAF1004001
- removed joint PAF1003500--PAF1003600
- removed joint PAF1003600--PAF1003700
- added joint 1_A--PAF1003600: type fixed, parent 1_A, child PAF1003600, origin xyz=0.0064 0.0129326 0.0275 rpy=1.04719714741 1.57079632679 0, axis 1.0 0.0 1.11022302463e-16
- added joint 1_A--PAF1003700: type fixed, parent 1_A, child PAF1003700, origin xyz=0.00409999738364 -0.00022020930368 -0.00208128063487 rpy=1.51319995882 0 -1.92248358723e-07, axis 8.10671871038e-09 -0.999999773716 -2.05797691055e-08
- added joint PAF1003500--PAF1003901: type fixed, parent PAF1003500, child PAF1003901, origin xyz=0.00501112 0.00642236 -0.031 rpy=2.77507338117 1.57079632679 0
- added joint PAF1003600--PAF1004001: type fixed, parent PAF1003600, child PAF1004001, origin xyz=-0.010973824593 -0.0237500416593 0.0027448885293 rpy=2.89289229734e-07 0.0108849789956 2.60776268803e-07
- joint PAF1002300--PAF1002500: limit (none) -> lower=-2.61799387799 upper=0.705631162427 effort=300 velocity=1; type continuous -> revolute
- joint PAF1002500--CUTOUT: limit (none) -> lower=-2.61799387799 upper=0.705631162427 effort=300 velocity=1; type continuous -> revolute
- joint PAF1003400--PAF1003801: type continuous -> fixed
- joint PAF1003700--PAF1004101: type continuous -> fixed
- joint PAF1003801--PAF1004201: limit (none) -> lower=-2.61799387799 upper=0.705631162427 effort=300 velocity=1; type continuous -> revolute
- joint PAF1003901--PAF1004301: limit (none) -> lower=-2.61799387799 upper=0.705631162427 effort=300 velocity=1; type continuous -> revolute
- joint PAF1004001--PAF1004201: limit (none) -> lower=-2.61799387799 upper=0.705631162427 effort=300 velocity=1; type continuous -> revolute
- joint PAF1004101--PAF1004401: limit (none) -> lower=-2.61799387799 upper=0.705631162427 effort=300 velocity=1; type continuous -> revolute
- joint PAF1004201--PAF1004500: limit (none) -> lower=-2.61799387799 upper=0.705631162427 effort=300 velocity=1; type continuous -> revolute
- joint PAF1004201--PAF10045000: limit (none) -> lower=-2.61799387799 upper=0.705631162427 effort=300 velocity=1; type continuous -> revolute
- joint PAF1004301--PAF1004600: limit (none) -> lower=-2.61799387799 upper=0.705631162427 effort=300 velocity=1; type continuous -> revolute
- joint PAF1004401--PAF1004700: limit (none) -> lower=-2.61799387799 upper=0.705631162427 effort=300 velocity=1; type continuous -> revolute
