Commit message: hanes hand with one finger

File: advr_mob_plt_description/urdf/test.urdf (robot description, URDF)
Before this commit: robot COVER, 6 links, 5 joints
Links:
- added link PAF1003801, mass 0.103446; collision mesh filename=package://advr_mob_plt_description/urdf/meshes/paf1003801_p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; visual mesh filename=package://advr_mob_plt_description/urdf/meshes/paf1003801_p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
- added link PAF1004201, mass 0.0118295; collision mesh filename=package://advr_mob_plt_description/urdf/meshes/paf1004201_p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; visual mesh filename=package://advr_mob_plt_description/urdf/meshes/paf1004201_p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
- added link PAF1004500, mass 0.190202; collision mesh filename=package://advr_mob_plt_description/urdf/meshes/paf1004500_p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; visual mesh filename=package://advr_mob_plt_description/urdf/meshes/paf1004500_p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
- added link PAF1004800, mass 0.00137117; collision mesh filename=package://advr_mob_plt_description/urdf/meshes/paf1004800_p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; visual mesh filename=package://advr_mob_plt_description/urdf/meshes/paf1004800_p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
Joints:
- added joint PAF1003400--PAF1003801: type fixed, parent PAF1003400, child PAF1003801, origin xyz=0 0 -9 rpy=1.58824971908 0 0, axis 0.0 -1.00000044025 -1.13856436057e-07
- added joint PAF1003801--PAF1004201: type revolute, parent PAF1003801, child PAF1004201, origin xyz=10.5 10.5 0 rpy=1.61820653951 1.57079602112 1.56584662577, axis 1.00000044025 -1.91634382918e-07 8.52805280907e-09, limit lower=-0.61 upper=0.705631162427 effort=300 velocity=1
- added joint PAF1004201--PAF1004500: type revolute, parent PAF1004201, child PAF1004500, origin xyz=0 1 33.5 rpy=-2.68780710036 2.39771271023e-07 0, axis -1.00000044025 -6.51257134887e-08 3.08022348461e-07, limit lower=-1.15 upper=0.02 effort=300 velocity=1
- added joint PAF1004500--PAF1004800: type fixed, parent PAF1004500, child PAF1004800, origin xyz=0 -1.5 -35 rpy=0 3.14159 3.14159

Commit message: hannes hand with four finger and extra shit

File: advr_mob_plt_description/urdf/test.urdf (robot description, URDF)
Before this commit: robot COVER, 10 links, 9 joints
Links:
- removed link PAF1003400
- removed link PAF1003500
- removed link PAF1003600
- removed link PAF1003700
- removed link PAF1003801
- removed link PAF1004201
- removed link PAF1004500
- removed link PAF1004800
- added link index_distal_link, mass 0.00137117; collision mesh filename=package://advr_mob_plt_description/urdf/meshes/paf1004800_p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; visual mesh filename=package://advr_mob_plt_description/urdf/meshes/paf1004800_p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
- added link index_medial_link, mass 0.190202; collision mesh filename=package://advr_mob_plt_description/urdf/meshes/paf1004500_p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; visual mesh filename=package://advr_mob_plt_description/urdf/meshes/paf1004500_p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
- added link index_mount_1_link, mass 0.0532202; collision mesh filename=package://advr_mob_plt_description/urdf/meshes/paf1003400_p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; visual mesh filename=package://advr_mob_plt_description/urdf/meshes/paf1003400_p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
- added link index_mount_2_link, mass 0.103446; collision mesh filename=package://advr_mob_plt_description/urdf/meshes/paf1003801_p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; visual mesh filename=package://advr_mob_plt_description/urdf/meshes/paf1003801_p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
- added link index_proximal_link, mass 0.0118295; collision mesh filename=package://advr_mob_plt_description/urdf/meshes/paf1004201_p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; visual mesh filename=package://advr_mob_plt_description/urdf/meshes/paf1004201_p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
- added link lil_distal_link, mass 0.000756894; collision mesh filename=package://advr_mob_plt_description/urdf/meshes/paf1005000_p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; visual mesh filename=package://advr_mob_plt_description/urdf/meshes/paf1005000_p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
- added link lil_medial_link, mass 0.0408908; collision mesh filename=package://advr_mob_plt_description/urdf/meshes/paf1004700_p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; visual mesh filename=package://advr_mob_plt_description/urdf/meshes/paf1004700_p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
- added link lil_mount_1_link, mass 0.012343; collision mesh filename=package://advr_mob_plt_description/urdf/meshes/paf1003700_p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; visual mesh filename=package://advr_mob_plt_description/urdf/meshes/paf1003700_p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
- added link lil_mount_2_link, mass 0.0285302; collision mesh filename=package://advr_mob_plt_description/urdf/meshes/paf1004101_p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; visual mesh filename=package://advr_mob_plt_description/urdf/meshes/paf1004101_p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
- added link lil_proximal_link, mass 0.0032677; collision mesh filename=package://advr_mob_plt_description/urdf/meshes/paf1004401_p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; visual mesh filename=package://advr_mob_plt_description/urdf/meshes/paf1004401_p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
- added link middle_distal_link, mass 0.00168109; collision mesh filename=package://advr_mob_plt_description/urdf/meshes/paf1004900_p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; visual mesh filename=package://advr_mob_plt_description/urdf/meshes/paf1004900_p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
- added link middle_medial_link, mass 0.221705; collision mesh filename=package://advr_mob_plt_description/urdf/meshes/paf1004600_p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; visual mesh filename=package://advr_mob_plt_description/urdf/meshes/paf1004600_p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
- added link middle_mount_1_link, mass 0.0178762; collision mesh filename=package://advr_mob_plt_description/urdf/meshes/paf1003500_p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; visual mesh filename=package://advr_mob_plt_description/urdf/meshes/paf1003500_p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
- added link middle_mount_2_link, mass 0.100064; collision mesh filename=package://advr_mob_plt_description/urdf/meshes/paf1003901_p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; visual mesh filename=package://advr_mob_plt_description/urdf/meshes/paf1003901_p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
- added link middle_proximal_link, mass 0.332988; collision mesh filename=package://advr_mob_plt_description/urdf/meshes/paf1004301_p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; visual mesh filename=package://advr_mob_plt_description/urdf/meshes/paf1004301_p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
- added link ring_distal_link, mass 0.00137117; collision mesh filename=package://advr_mob_plt_description/urdf/meshes/paf1004800_p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; visual mesh filename=package://advr_mob_plt_description/urdf/meshes/paf1004800_p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
- added link ring_medial_link, mass 0.190202; collision mesh filename=package://advr_mob_plt_description/urdf/meshes/paf1004500_p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; visual mesh filename=package://advr_mob_plt_description/urdf/meshes/paf1004500_p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
- added link ring_mount_1_link, mass 0.0185208; collision mesh filename=package://advr_mob_plt_description/urdf/meshes/paf1003600_p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; visual mesh filename=package://advr_mob_plt_description/urdf/meshes/paf1003600_p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
- added link ring_mount_2_link, mass 0.0996106; collision mesh filename=package://advr_mob_plt_description/urdf/meshes/paf1004001_p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; visual mesh filename=package://advr_mob_plt_description/urdf/meshes/paf1004001_p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
- added link ring_proximal_link, mass 0.0118295; collision mesh filename=package://advr_mob_plt_description/urdf/meshes/paf1004201_p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; visual mesh filename=package://advr_mob_plt_description/urdf/meshes/paf1004201_p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
Joints:
- removed joint 1_A--PAF1003400
- removed joint 1_A--PAF1003500
- removed joint 1_A--PAF1003600
- removed joint 1_A__PAF1003700
- removed joint PAF1003400--PAF1003801
- removed joint PAF1003801--PAF1004201
- removed joint PAF1004201--PAF1004500
- removed joint PAF1004500--PAF1004800
- added joint index_medial_distal_joint: type fixed, parent index_medial_link, child index_distal_link, origin xyz=0 -1.5 -35 rpy=0 3.14159 3.14159
- added joint index_mount_joint: type fixed, parent index_mount_1_link, child index_mount_2_link, origin xyz=0 0 -9 rpy=1.58824971908 0 0, axis 0.0 -1.00000044025 -1.13856436057e-07
- added joint index_mount_proximal_joint: type revolute, parent index_mount_2_link, child index_proximal_link, origin xyz=10.5 10.5 0 rpy=1.61820653951 1.57079602112 1.56584662577, axis 1.00000044025 -1.91634382918e-07 8.52805280907e-09, limit lower=-0.61 upper=0.705631162427 effort=300 velocity=1
- added joint index_proximal_medial_joint: type revolute, parent index_proximal_link, child index_medial_link, origin xyz=0 1 33.5 rpy=-2.68780710036 2.39771271023e-07 0, axis -1.00000044025 -6.51257134887e-08 3.08022348461e-07, limit lower=-1.15 upper=0.02 effort=300 velocity=1
- added joint lil_medial_distal: type fixed, parent lil_medial_link, child lil_distal_link, origin xyz=0 -1.5 -35 rpy=0 3.14159 3.14159
- added joint lil_mount_joint: type fixed, parent lil_mount_1_link, child lil_mount_2_link, origin xyz=0 0 -9 rpy=1.58824971908 0 0, axis 8.10671871038e-09 -0.999999773716 -2.05797691055e-08
- added joint lil_mount_proximal_joint: type revolute, parent lil_mount_2_link, child lil_proximal_link, origin xyz=10.5 10.5 0 rpy=1.61820653951 1.57079602112 1.56584662577, axis 0.999999678896 1.99802328055e-08 2.77878688046e-08, limit lower=-0.27 upper=0.705631162427 effort=300 velocity=1
- added joint lil_proximal_medial_joint: type revolute, parent lil_proximal_link, child lil_medial_link, origin xyz=0 1 29.5 rpy=-2.68780710036 2.39771271023e-07 0, axis -0.999999678896 -1.31398492954e-08 3.17077668288e-09, limit lower=-0.60 upper=0.71 effort=300 velocity=1
- added joint middle_medial_distal_joint: type fixed, parent middle_medial_link, child middle_distal_link, origin xyz=0 -1.5 -35 rpy=0 3.14159 3.14159
- added joint middle_mount_joint: type fixed, parent middle_mount_1_link, child middle_mount_2_link, origin xyz=0 0 -9 rpy=1.58824971908 0 0
- added joint middle_mount_proximal_joint: type revolute, parent middle_mount_2_link, child middle_proximal_link, origin xyz=10.5 10.5 0 rpy=1.61820653951 1.57079602112 1.56584662577, axis 0.999999619912 -8.81751169857e-08 2.40175518709e-08, limit lower=-0.66 upper=0.705631162427 effort=300 velocity=1
- added joint middle_proximal_medial_joint: type revolute, parent middle_proximal_link, child middle_medial_link, origin xyz=0 1 36.5 rpy=-2.68780710036 2.39771271023e-07 0, axis -0.999999619912 1.24171011417e-07 2.37297750894e-07, limit lower=0.08 upper=-1.18 effort=300 velocity=1
- added joint palm_index_mount_joint: type fixed, parent 1_A, child index_mount_1_link, origin xyz=29 10 -28 rpy=1.57 1.57 0.436332
- added joint palm_lil_mount_joint: type fixed, parent 1_A, child lil_mount_1_link, origin xyz=-36 -6 -20 rpy=1.57 1.57 -0.261799, axis 8.10671871038e-09 -0.999999773716 -2.05797691055e-08
- added joint palm_middle_mount_joint: type fixed, parent 1_A, child middle_mount_1_link, origin xyz=10 -3 -32 rpy=1.57 1.57 0.261799, axis 1.0 0.0 1.11022302463e-16
- added joint palm_ring_mount_joint: type fixed, parent 1_A, child ring_mount_1_link, origin xyz=-12 -5 -30 rpy=1.57 1.57 -0.174533
- added joint ring_medial_distal_joint: type fixed, parent ring_medial_link, child ring_distal_link, origin xyz=0 -1.5 -35 rpy=0 3.14159 3.14159
- added joint ring_mount_joint: type fixed, parent ring_mount_1_link, child ring_mount_2_link, origin xyz=0 0 -9 rpy=1.58824971908 0 0
- added joint ring_mount_proximal_joint: type revolute, parent ring_mount_2_link, child ring_proximal_link, origin xyz=10.5 10.5 0 rpy=1.61820653951 1.57079602112 1.56584662577, axis 1.00000024783 2.36992810717e-07 -1.72229714934e-08, limit lower=-0.42 upper=0.705631162427 effort=300 velocity=1
- added joint ring_proximal_medial_joint: type revolute, parent ring_proximal_link, child ring_medial_link, origin xyz=0 1 33 rpy=-2.68780710036 2.39771271023e-07 0, axis -1.00000024783 -1.20997757813e-07 9.61299631563e-08, limit lower=-0.61 upper=0.705631162427 effort=300 velocity=1

Commit message: approx joint limits and  mount_1 axis orientation corrected to avoid collision

File: advr_mob_plt_description/urdf/test.urdf (robot description, URDF)
Before this commit: robot COVER, 22 links, 21 joints
Joints:
- joint index_mount_proximal_joint: limit lower=-0.61 upper=0.705631162427 effort=300 velocity=1 -> lower=0.14 upper=0.705631162427 effort=300 velocity=1
- joint middle_mount_proximal_joint: limit lower=-0.66 upper=0.705631162427 effort=300 velocity=1 -> lower=0.04 upper=0.705631162427 effort=300 velocity=1
- joint palm_index_mount_joint: origin xyz=29 10 -28 rpy=1.57 1.57 0.436332 -> xyz=29 10 -28 rpy=1.57 1.57 -0.001
- joint palm_middle_mount_joint: origin xyz=10 -3 -32 rpy=1.57 1.57 0.261799 -> xyz=10 -3 -32 rpy=1.57 1.57 0
- joint palm_ring_mount_joint: origin xyz=-12 -5 -30 rpy=1.57 1.57 -0.174533 -> xyz=-12 -5 -30 rpy=1.57 1.57 0
- joint ring_mount_proximal_joint: limit lower=-0.42 upper=0.705631162427 effort=300 velocity=1 -> lower=0.14 upper=0.705631162427 effort=300 velocity=1
- joint ring_proximal_medial_joint: limit lower=-0.61 upper=0.705631162427 effort=300 velocity=1 -> lower=-0.61 upper=0.13 effort=300 velocity=1

Commit message: thumb joint 1 approximated

File: advr_mob_plt_description/urdf/test.urdf (robot description, URDF)
Before this commit: robot COVER, 22 links, 21 joints
Links:
- added link PAF1002300, mass 48784.5; collision mesh filename=package://advr_mob_plt_description/urdf/meshes/paf1002300_p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; visual mesh filename=package://advr_mob_plt_description/urdf/meshes/paf1002300_p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
- added link PAF1002500, mass 0.0602771; collision mesh filename=package://advr_mob_plt_description/urdf/meshes/paf1002500_p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; visual mesh filename=package://advr_mob_plt_description/urdf/meshes/paf1002500_p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
Joints:
- added joint 1_A--PAF1002300: type fixed, parent 1_A, child PAF1002300, origin xyz=20 12 5 rpy=-0.123389636399 0.0215437373873 0.976908191421
- added joint PAF1002300__PAF1002500: type fixed, parent PAF1002300, child PAF1002500, origin xyz=3 2.5 0 rpy=0 0 0, axis -1.0000001741 4.77024647005e-07 2.31302308709e-07

Commit message: approximated hand with joint limits but unnecessary extra meshes appear

File: advr_mob_plt_description/urdf/test.urdf (robot description, URDF)
Before this commit: robot COVER, 24 links, 23 joints
Links:
- added link CUTOUT, mass 179552000.0; collision mesh filename=package://advr_mob_plt_description/urdf/meshes/cutout_asm-b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; visual mesh filename=package://advr_mob_plt_description/urdf/meshes/cutout_asm-b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
Joints:
- added joint PAF1002500__CUTOUT: type revolute, parent PAF1002500, child CUTOUT, origin xyz=16 16 24 rpy= 0 0 -0.785398, axis 1.00000033972 1.92759832931e-08 -1.39895338369e-08, limit lower=-0.72 upper=0.705631162427 effort=300 velocity=1

Commit message: urdf joint and link naming done

File: advr_mob_plt_description/urdf/test.urdf (robot description, URDF)
Before this commit: robot COVER, 25 links, 24 joints
Links:
- removed link CUTOUT
- removed link PAF1002300
- removed link PAF1002500
- added link thumb_distal_link, mass 179552000.0; collision mesh filename=package://advr_mob_plt_description/urdf/meshes/cutout_asm-b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; visual mesh filename=package://advr_mob_plt_description/urdf/meshes/cutout_asm-b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
- added link thumb_medial_link, mass 0.0602771; collision mesh filename=package://advr_mob_plt_description/urdf/meshes/paf1002500_p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; visual mesh filename=package://advr_mob_plt_description/urdf/meshes/paf1002500_p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
- added link thumb_mount_link, mass 48784.5; collision mesh filename=package://advr_mob_plt_description/urdf/meshes/paf1002300_p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; visual mesh filename=package://advr_mob_plt_description/urdf/meshes/paf1002300_p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
Joints:
- removed joint 1_A--PAF1002300
- removed joint PAF1002300__PAF1002500
- removed joint PAF1002500__CUTOUT
- added joint palm_thumb_mount_joint: type fixed, parent 1_A, child thumb_mount_link, origin xyz=20 12 5 rpy=-0.123389636399 0.0215437373873 0.976908191421
- added joint thumb_medial_distal_joint: type revolute, parent thumb_medial_link, child thumb_distal_link, origin xyz=16 16 24 rpy= 0 0 -0.785398, axis 1.00000033972 1.92759832931e-08 -1.39895338369e-08, limit lower=-0.72 upper=0.705631162427 effort=300 velocity=1
- added joint thumb_mount_medial_joint: type fixed, parent thumb_mount_link, child thumb_medial_link, origin xyz=3 2.5 0 rpy=0 0 0, axis -1.0000001741 4.77024647005e-07 2.31302308709e-07
